File: 01 - Board/KiCad/screen.kicad_sch (KiCad schematic)
At the start: 15 parts, among them J1 OLED UG-9616TSWCG02, SW1 SW_Push

Commit message: PCB order
Parts:
- added C2 (x2): 1u, Capacitor_SMD:C_0603_1608Metric_Pad1.08x0.95mm_HandSolder, symbol Device:C
- added R1 (x2): 2k4, Resistor_SMD:R_0603_1608Metric_Pad0.98x0.95mm_HandSolder, symbol Device:R_US
- added SW2, SW3: SW_Push, symbol Switch:SW_Push
Connections:
- net +3V3: now also R1.1, R1.1
- net GND: now also C2.2, C2.2, SW2.2, SW3.2
- new net BTN_LEFT: C2.1, R1.2, SW2.1
- new net BTN_RIGHT: C2.1, R1.2, SW3.1
Other:
- note added: "CONTROL BUTTONS"
- moved on the sheet: C2, R1, SW1
