File: 01 - Board/KiCad/HotPlate.kicad_pcb (KiCad board)
At the start: 2 copper layers, 220 x 120 mm, 29 parts, among them J1 OLED UG-9616TSWCG02, J2 USB_C_Receptacle_PowerOnly_6P, Q1 2N7002, U1 CYPD3177, U2 IRF9358TRPBF

Commit message: PCB order
Parts:
- removed C2: C, Capacitor_SMD:C_0603_1608Metric_Pad1.08x0.95mm_HandSolder
- removed C4: 100n, Capacitor_SMD:C_0603_1608Metric_Pad1.08x0.95mm_HandSolder
- removed C5, C7: 1uF, Capacitor_SMD:C_0603_1608Metric_Pad1.08x0.95mm_HandSolder
- removed J1: OLED UG-9616TSWCG02, Footprints:UG-9616TSWCG02
- added ?: , , F.Cu at (251.0, 54.0)
- added ?: , , F.Cu at (245.0, 39.0)
- added C101: 10u, Capacitor_SMD:CP_Elec_4x5.4, F.Cu at (47.6, 46.5)
- added C103: 1u, Capacitor_SMD:C_0603_1608Metric_Pad1.08x0.95mm_HandSolder, F.Cu at (60.4, 51.3)
- added C109: 100n, Capacitor_SMD:C_1210_3225Metric_Pad1.33x2.70mm_HandSolder, F.Cu at (77.8, 54.9)
- added C201: 4u7, Capacitor_SMD:C_0805_2012Metric_Pad1.18x1.45mm_HandSolder, F.Cu at (133.5, 37.9)
- added C202: 100n, Capacitor_SMD:C_0603_1608Metric_Pad1.08x0.95mm_HandSolder, F.Cu at (132.6, 44.0)
- added C203: 4u7, Capacitor_SMD:C_0805_2012Metric_Pad1.18x1.45mm_HandSolder, F.Cu at (137.0, 46.3)
- added C204: 100n, Capacitor_SMD:C_0603_1608Metric_Pad1.08x0.95mm_HandSolder, F.Cu at (130.1, 41.1)
- added C205: 4u7, Capacitor_SMD:C_0805_2012Metric_Pad1.18x1.45mm_HandSolder, F.Cu at (137.0, 44.0)
- added C206: 100n, Capacitor_SMD:C_0603_1608Metric_Pad1.08x0.95mm_HandSolder, F.Cu at (96.6, 44.7)
- added C207: 100n, Capacitor_SMD:C_0603_1608Metric_Pad1.08x0.95mm_HandSolder, F.Cu at (99.3, 41.7)
- added C208: 4u7, Capacitor_SMD:C_0805_2012Metric_Pad1.18x1.45mm_HandSolder, F.Cu at (97.8, 40.2)
- added C301: 1u, Capacitor_SMD:C_0603_1608Metric_Pad1.08x0.95mm_HandSolder, F.Cu at (220.0, 48.0)
- added C302: 1u, Capacitor_SMD:C_0603_1608Metric_Pad1.08x0.95mm_HandSolder, F.Cu at (210.0, 48.0)
- added C303: 1u, Capacitor_SMD:C_0603_1608Metric_Pad1.08x0.95mm_HandSolder, F.Cu at (200.0, 48.0)
- added C304: 1u, Capacitor_SMD:C_0603_1608Metric_Pad1.08x0.95mm_HandSolder, F.Cu at (153.4, 42.3)
- added C305: 1u, Capacitor_SMD:C_0603_1608Metric_Pad1.08x0.95mm_HandSolder, F.Cu at (153.4, 40.5)
- added C306: 1u, Capacitor_SMD:C_0603_1608Metric_Pad1.08x0.95mm_HandSolder, F.Cu at (157.1, 49.6)
- added C307: 1u, Capacitor_SMD:C_0603_1608Metric_Pad1.08x0.95mm_HandSolder, F.Cu at (157.1, 47.9)
- added C308: 1u, Capacitor_SMD:C_0603_1608Metric_Pad1.08x0.95mm_HandSolder, F.Cu at (158.2, 36.2)
- added C309: 1u, Capacitor_SMD:C_0603_1608Metric_Pad1.08x0.95mm_HandSolder, F.Cu at (154.3, 37.8)
- added C310: 4u7, Capacitor_SMD:C_0805_2012Metric_Pad1.18x1.45mm_HandSolder, F.Cu at (153.9, 48.5)
- added C401: 100n, Capacitor_SMD:C_0603_1608Metric_Pad1.08x0.95mm_HandSolder, F.Cu at (238.4, 49.0)
- added C402: 100n, Capacitor_SMD:C_0603_1608Metric_Pad1.08x0.95mm_HandSolder, F.Cu at (241.2, 52.1)
- added D101: RED, LED_SMD:LED_0603_1608Metric_Pad1.05x0.95mm_HandSolder, F.Cu at (80.7, 41.2)
- added D102: D_Schottky, Diode_SMD:D_SMA, F.Cu at (77.8, 51.1)
- added D201: RED, LED_SMD:LED_0603_1608Metric_Pad1.05x0.95mm_HandSolder, F.Cu at (141.7, 44.3)
- added D202: RED, LED_SMD:LED_0603_1608Metric_Pad1.05x0.95mm_HandSolder, F.Cu at (109.8, 39.0)
- added D203: D_Schottky, Diode_SMD:D_SOD-323_HandSoldering, F.Cu at (120.9, 39.4)
- added FID1: Fiducial_0.5mm_Mask1mm, Fiducial:Fiducial_0.5mm_Mask1mm, F.Cu at (40.0, 50.0)
- added G***: LOGO, LOGO, F.Cu at (145.0, 98.0)
- added J201: Conn_ARM_SWD_TagConnect_TC2030, Connector:Tag-Connect_TC2030-IDC-FP_2x03_P1.27mm_Vertical, F.Cu at (115.0, 41.6)
- added J301: OLED UG-9616TSWCG02, Footprints:UG-9616TSWCG02, F.Cu at (157.3, 42.0)
- added L201: 10u, Footprints:L_4.2x4.4_H2, F.Cu at (138.4, 39.8)
- added Q102: NMOS_ALT, Package_TO_SOT_SMD:TO-252-2, F.Cu at (87.2, 51.9)
- added R102: 5k1, Resistor_SMD:R_0603_1608Metric_Pad0.98x0.95mm_HandSolder, F.Cu at (74.5, 41.2)
- added R108: 1k, Resistor_SMD:R_0603_1608Metric_Pad0.98x0.95mm_HandSolder, F.Cu at (66.7, 45.2)
- added R110: 150, Resistor_SMD:R_0805_2012Metric_Pad1.20x1.40mm_HandSolder, F.Cu at (98.1, 53.1)
- added R118: 5k1, Resistor_SMD:R_0603_1608Metric_Pad0.98x0.95mm_HandSolder, F.Cu at (73.5, 45.2)
- added R119: 0, Resistor_SMD:R_0603_1608Metric_Pad0.98x0.95mm_HandSolder, F.Cu at (75.2, 45.2)
- added R201: 10k, Resistor_SMD:R_0603_1608Metric_Pad0.98x0.95mm_HandSolder, F.Cu at (130.1, 36.9)
- added R202: 10k, Resistor_SMD:R_0603_1608Metric_Pad0.98x0.95mm_HandSolder, F.Cu at (127.5, 37.8)
- added R203: 33k, Resistor_SMD:R_0603_1608Metric_Pad0.98x0.95mm_HandSolder, F.Cu at (126.7, 41.1)
- added R204: 10k, Resistor_SMD:R_0603_1608Metric_Pad0.98x0.95mm_HandSolder, F.Cu at (128.4, 41.1)
- added R205: 1k, Resistor_SMD:R_0603_1608Metric_Pad0.98x0.95mm_HandSolder, F.Cu at (142.6, 47.2)
- added R206: 1k, Resistor_SMD:R_0603_1608Metric_Pad0.98x0.95mm_HandSolder, F.Cu at (109.8, 42.5)
- added R301: 2k2, Resistor_SMD:R_0603_1608Metric_Pad0.98x0.95mm_HandSolder, F.Cu at (220.0, 50.0)
- added R302: 2k2, Resistor_SMD:R_0603_1608Metric_Pad0.98x0.95mm_HandSolder, F.Cu at (210.0, 50.0)
- added R303: 2k2, Resistor_SMD:R_0603_1608Metric_Pad0.98x0.95mm_HandSolder, F.Cu at (200.0, 50.0)
- added R304: 2k2, Resistor_SMD:R_0603_1608Metric_Pad0.98x0.95mm_HandSolder, F.Cu at (162.2, 47.9)
- added R305: 2k2, Resistor_SMD:R_0603_1608Metric_Pad0.98x0.95mm_HandSolder, F.Cu at (112.1, 49.2)
- added R306: 2k2, Resistor_SMD:R_0603_1608Metric_Pad0.98x0.95mm_HandSolder, F.Cu at (112.1, 50.9)
- added R307: 820k, Resistor_SMD:R_0603_1608Metric_Pad0.98x0.95mm_HandSolder, F.Cu at (153.4, 45.4)
- added R401: 280, Resistor_SMD:R_0603_1608Metric_Pad0.98x0.95mm_HandSolder, F.Cu at (244.0, 48.7)
- added R402: 8k2, Resistor_SMD:R_0603_1608Metric_Pad0.98x0.95mm_HandSolder, F.Cu at (241.2, 44.0)
- added R403: 5k4, Resistor_SMD:R_0603_1608Metric_Pad0.98x0.95mm_HandSolder, F.Cu at (241.2, 45.8)
- added R404: 1k5, Resistor_SMD:R_0603_1608Metric_Pad0.98x0.95mm_HandSolder, F.Cu at (236.6, 49.0)
- added REF**: MountingHole_3.5mm, MountingHole:MountingHole_3.5mm, F.Cu at (39.0, 39.0)
- added REF**: MountingHole_3.5mm, MountingHole:MountingHole_3.5mm, F.Cu at (39.0, 151.0)
- added REF**: OSHW-Logo2_7.3x6mm_SilkScreen, Symbol:OSHW-Logo2_7.3x6mm_SilkScreen, F.Cu at (250.8, 129.6)
- added REF**: MountingHole_3.5mm, MountingHole:MountingHole_3.5mm, F.Cu at (145.0, 39.0)
- added REF**: MountingHole_3.5mm, MountingHole:MountingHole_3.5mm, F.Cu at (251.0, 151.0)
- added REF**: MountingHole_3.5mm, MountingHole:MountingHole_3.5mm, F.Cu at (251.0, 39.0)
- added SW301: SW_Push, Footprints:SW_Push_1P1T_NO_3.5x8mm_H3mm, F.Cu at (220.0, 42.0)
- added SW302: SW_Push, Footprints:SW_Push_1P1T_NO_3.5x8mm_H3mm, F.Cu at (210.0, 42.0)
- added SW303: SW_Push, Footprints:SW_Push_1P1T_NO_3.5x8mm_H3mm, F.Cu at (200.0, 42.0)
- added TH401: Thermistor_NTC, Connector_PinHeader_2.54mm:PinHeader_2x01_P2.54mm_Vertical, F.Cu at (249.5, 47.8)
- added TP201: TestPoint_2Pole, Footprints:TestPoint_Pad_D1.0mm_DUAL, F.Cu at (139.8, 47.8)
- added U201: AP62300TWU, Package_TO_SOT_SMD:TSOT-23-6, F.Cu at (133.4, 41.1)
- added U202: STM32G030K8T6, Package_QFP:LQFP-32_7x7mm_P0.8mm, F.Cu at (104.0, 46.5)
- added U401: LM321LV, Package_TO_SOT_SMD:SOT-23-5, F.Cu at (241.2, 49.0)
- added kibuzzard-64D50818: G***, kibuzzard-64D50818, F.Cu at (54.5, 44.0)
- added kibuzzard-64D5083A: G***, kibuzzard-64D5083A, F.Cu at (116.7, 36.3)
- added kibuzzard-64D50885: G***, kibuzzard-64D50885, F.Cu at (174.4, 49.9)
- added kibuzzard-64D508C0: G***, kibuzzard-64D508C0, F.Cu at (219.9, 36.4)
- added kibuzzard-64D508E0: G***, kibuzzard-64D508E0, F.Cu at (210.0, 36.4)
- added kibuzzard-64D508EC: G***, kibuzzard-64D508EC, F.Cu at (200.0, 36.3)
- added kibuzzard-64D5DE4F: G***, kibuzzard-64D5DE4F, F.Cu at (145.1, 44.4)
- added kibuzzard-64D5DEAF: G***, kibuzzard-64D5DEAF, F.Cu at (87.0, 41.2)
- added kibuzzard-64D5E8FE: G***, kibuzzard-64D5E8FE, F.Cu at (248.3, 45.1)
- C102: renamed from C6; value 1uF -> 4u7; footprint Capacitor_SMD:C_0603_1608Metric_Pad1.08x0.95mm_HandSolder -> Capacitor_SMD:C_0805_2012Metric_Pad1.18x1.45mm_HandSolder
- C104: renamed from C8; value 1uF -> 1u
- C105: renamed from C9; value 1uF -> 1u
- C106: renamed from C1; value 1uF -> 1u
- C107: renamed from C2; value 1uF -> 100n
- R101: renamed from R2; value 2k4 -> 1k
- R103: renamed from R1; value 2k4 -> 2k2
- R104: renamed from R12; value 2k4 -> 2k2
- R105: renamed from R14; value 5k1 -> 2k2
- R106: renamed from R11; value 2k4 -> 5k1
- R107: renamed from R13; value 2k4 -> 2k2
- R109: renamed from R3; value 5k1 -> 2k2
- R111: renamed from R4; value 2k4 -> 5k1
- R113: renamed from R6; value 2k4 -> 2k2
- R115: renamed from R8; value 5k1 -> 2k2
- R117: renamed from R10; value 0 -> 5k1
- moved R105 83.1 mm to (106.2, 39.2), turned to 180 degrees
- moved R104 77.1 mm to (101.8, 39.2), turned to 45 degrees
- moved R103 74.3 mm to (95.7, 47.4), turned to 180 degrees
- moved R107 68.9 mm to (95.7, 49.1), turned to 180 degrees
- moved R101 66.5 mm to (83.1, 41.2), turned to 90 degrees
- moved Q101 53.9 mm to (77.6, 41.2)
- moved C107 49.1 mm to (63.5, 39.6), turned to 90 degrees
- moved C108 49.0 mm to (61.8, 39.6), turned to 90 degrees
- moved C104 46.9 mm to (70.1, 52.4), turned to 90 degrees
- moved C105 45.8 mm to (60.1, 39.6), turned to 90 degrees
- moved C102 35.4 mm to (47.3, 50.8), turned to 180 degrees
- moved R111 35.2 mm to (87.2, 44.4), turned to 180 degrees
- moved R106 34.9 mm to (62.2, 51.3), turned to 90 degrees
- moved R117 24.1 mm to (70.1, 45.2), turned to -90 degrees
- moved R116 23.9 mm to (71.8, 45.2), turned to 90 degrees
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- renumbered C3 to C108, J2 to J101, Q1 to Q101, R5 to R112, R7 to R114, R9 to R116, U2 to U101, U1 to U102
Connections:
- net Net-(J2-CC1) renamed /CC1
- net Net-(J2-CC2) renamed /CC2
- net Net-(Q1-G) renamed /LED_FAULT
- C102 pad 1: Net-(U1-VBUS_IN) -> VBUS
- C104 pad 1: Net-(U1-VBUS_IN) -> /BUS_HEATSINK
- C104 pad 2: Net-(U2A-G1) -> Net-(U101A-G1)
- C105 pad 1: Net-(U2B-S2) -> VDD
- C105 pad 2: Net-(U2A-G1) -> GND
- C106 pad 1: VDD -> +1V8
- C107 pad 1: +1V8 -> VDD
- J101 pad A9: Net-(U1-VBUS_IN) -> VBUS
- J101 pad B9: Net-(U1-VBUS_IN) -> VBUS
- R101 pad 1: VDD -> +3V3
- R103 pad 1: VDD -> +3V3
- R104 pad 1: VDD -> +3V3
- R105 pad 1: Net-(U1-VBUS_IN) -> +3V3
- R105 pad 2: Net-(U2A-G1) -> PD_SCL
- R106 pad 1: VDD -> VBUS
- R106 pad 2: PD_SCL -> Net-(U101A-G1)
- R107 pad 1: Net-(U2A-G1) -> +3V3
- R107 pad 2: Net-(R13-Pad2) -> PD_HPI
- R109 pad 1: VDD -> PD_SAFE
- R109 pad 2: Net-(U1-VBUS_MAX) -> /SAFE
- R111 pad 1: Net-(U1-VBUS_MAX) -> Net-(Q102-G)
- R112 pad 1: VDD -> +3V3
- R112 pad 2: Net-(U1-VBUS_MIN) -> /VBUS_MAX
- R113 pad 1: Net-(U1-VBUS_MIN) -> /VBUS_MAX
- R114 pad 1: VDD -> +3V3
- R114 pad 2: Net-(U1-ISNK_COARSE) -> /VBUS_MIN
- R115 pad 1: Net-(U1-ISNK_COARSE) -> /VBUS_MIN
- R116 pad 1: VDD -> +3V3
- R116 pad 2: Net-(U1-ISNK_FINE) -> /ISNK_COARSE
- R117 pad 1: Net-(U1-ISNK_FINE) -> /ISNK_COARSE
- U101 pad 1: Net-(U2B-S2) -> Net-(U101A-S1)
- U101 pad 2: Net-(U2A-G1) -> Net-(U101A-G1)
- U101 pad 3: Net-(U2A-S1) -> Net-(U101A-S1)
- U101 pad 4: Net-(U2A-G1) -> Net-(U101A-G1)
- U101 pad 5: Net-(U1-VBUS_IN) -> VBUS
- U101 pad 6: Net-(U1-VBUS_IN) -> VBUS
- U101 pad 7: Net-(U2A-S1) -> /BUS_HEATSINK
- U101 pad 8: Net-(U2A-S1) -> /BUS_HEATSINK
- U102 pad 1: Net-(U1-VBUS_MIN) -> /VBUS_MIN
- U102 pad 11: unconnected-(U1-VDC_OUT-Pad11) -> /BUS_HEATSINK
- U102 pad 18: Net-(U1-VBUS_IN) -> VBUS
- U102 pad 2: Net-(U1-VBUS_MAX) -> /VBUS_MAX
- U102 pad 3: Net-(R13-Pad2) -> /VBUS_EN
- U102 pad 4: unconnected-(U1-Pad4) -> /SAFE
- U102 pad 5: Net-(U1-ISNK_COARSE) -> /ISNK_COARSE
- U102 pad 6: Net-(U1-ISNK_FINE) -> /ISNK_FINE
Routing:
- net /BUS_HEATSINK: track 0.00 -> 14239.4 mm, vias 0 -> 2
- net +3V3: track 0.00 -> 295.8 mm, vias 0 -> 9
- net TEMP: track 0.00 -> 140.3 mm
- net BTN_OKEY: track 0.00 -> 121.3 mm
- net BTN_UP: track 0.00 -> 110.6 mm
- net BTN_DOWN: track 0.00 -> 99.9 mm
- net VBUS: track 0.00 -> 94.2 mm, vias 0 -> 2
- net ~{RSTn}_OLED: track 0.00 -> 67.0 mm
- net SCL_OLED: track 0.00 -> 63.5 mm
- net SDA_OLED: track 0.00 -> 51.6 mm
- net PD_SAFE: track 0.00 -> 43.1 mm
- net PD_SCL: track 0.00 -> 41.7 mm
- net PD_HPI: track 0.00 -> 39.1 mm
- net PD_SDA: track 0.00 -> 37.1 mm
- net PD_FLIP: track 0.00 -> 36.9 mm
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- added copper zone on B.Cu, net +3V3
- added copper zone on F.Cu, net +3V3
- added copper zone on F.Cu, net /BUS_HEATSINK
- added copper zone on F.Cu, net /MCU/SW
- added copper zone on B.Cu, net GND
- added copper zone on F.Cu, net GND
- added copper zone on F.Cu, net Net-(U101A-G1)
- added copper zone on F.Cu, net VBUS
Other:
- board text added: "CAUTION"
- board text added: "FID2"
- board text added: "FID3"
- board text added: "HOT PLATE A"
- board text added: "HOT SURFACE"
- board text added: "JLCJLCJLCJLC"
- board text added: "SERGIO IBARRA"

Commit message: Pedido
Parts:
- removed kibuzzard-64D5083A: G***, kibuzzard-64D5083A
- removed kibuzzard-64D508C0: G***, kibuzzard-64D508C0
- removed kibuzzard-64D508E0: G***, kibuzzard-64D508E0
- removed kibuzzard-64D508EC: G***, kibuzzard-64D508EC
- removed kibuzzard-64D5DE4F: G***, kibuzzard-64D5DE4F
- added kibuzzard-64D63906: G***, kibuzzard-64D63906, F.Cu at (116.3, 36.3)
- added kibuzzard-64D73B55: G***, kibuzzard-64D73B55, F.Cu at (200.0, 36.2)
- added kibuzzard-64D73B79: G***, kibuzzard-64D73B79, F.Cu at (210.0, 36.2)
- added kibuzzard-64D73B89: G***, kibuzzard-64D73B89, F.Cu at (219.9, 36.2)
- added kibuzzard-64D73C73: G***, kibuzzard-64D73C73, F.Cu at (144.9, 43.5)
- moved kibuzzard-64D50818 0.30 mm to (54.8, 44.0)
