File: 01 - Board/KiCad/HotPlate.kicad_sch (KiCad schematic)
At the start: 30 parts, among them J2 USB_C_Receptacle_PowerOnly_6P, Q1 2N7002, U1 CYPD3177, U2 IRF9358TRPBF

Commit message: PCB order
Parts:
- removed C5, C7: 1u, Capacitor_SMD:C_0603_1608Metric_Pad1.08x0.95mm_HandSolder, symbol Device:C
- added C101: 10u, Capacitor_SMD:CP_Elec_4x5.4, symbol Device:C_Polarized_US
- added C109: 100n, Capacitor_SMD:C_1210_3225Metric_Pad1.33x2.70mm_HandSolder, symbol Device:C
- added D102: D_Schottky, Diode_SMD:D_SMA, symbol Device:D_Schottky
- added Q102: NMOS_ALT, Package_TO_SOT_SMD:TO-252-2, symbol Symbols:NMOS_ALT
- added R107: 2k2, Resistor_SMD:R_0603_1608Metric_Pad0.98x0.95mm_HandSolder, symbol Device:R_US
- added R110: 150, Resistor_SMD:R_0805_2012Metric_Pad1.20x1.40mm_HandSolder, symbol Device:R_US
- added R111: 5k1, Resistor_SMD:R_0603_1608Metric_Pad0.98x0.95mm_HandSolder, symbol Device:R_US
- C102: renamed from C6; value 1u -> 4u7; footprint Capacitor_SMD:C_0603_1608Metric_Pad1.08x0.95mm_HandSolder -> Capacitor_SMD:C_0805_2012Metric_Pad1.18x1.45mm_HandSolder; LCSC Part # (none) -> C98195; MPN (none) -> CL21B475KAFNNNE
- C103: renamed from C8; LCSC Part # (none) -> C5673; MPN (none) -> CL10A105KA8NNNC
- C104: renamed from C9; LCSC Part # (none) -> C5673; MPN (none) -> CL10A105KA8NNNC; now not fitted
- C105: renamed from C1; LCSC Part # (none) -> C5673; MPN (none) -> CL10A105KA8NNNC
- C106: renamed from C2; LCSC Part # (none) -> C5673; MPN (none) -> CL10A105KA8NNNC
- C107: renamed from C3; LCSC Part # (none) -> C14663; MPN (none) -> CC0603KRX7R9BB104
- C108: renamed from C4; LCSC Part # (none) -> C14663; MPN (none) -> CC0603KRX7R9BB104
- D101: renamed from D1; value LED -> RED; footprint (none) -> LED_SMD:LED_0603_1608Metric_Pad1.05x0.95mm_HandSolder; LCSC Part # (none) -> C965799; MPN (none) -> XL-1608SURC-06
- J101: renamed from J2; LCSC Part # (none) -> C2764612; MPN (none) -> U262-061N-4BVC11
- Q101: renamed from Q1; LCSC Part # (none) -> C414015; MPN (none) -> 2N7002K
- R101: renamed from R2; LCSC Part # (none) -> C103209; MPN (none) -> RTT03102JTP
- R102: renamed from R15; LCSC Part # (none) -> C26000; MPN (none) -> 0603WAJ0512T5E
- R103: renamed from R1; value 2k4 -> 2k2; LCSC Part # (none) -> C2907117
- R104: renamed from R12; value 2k4 -> 2k2; LCSC Part # (none) -> C2907117
- R105: renamed from R11; value 2k4 -> 2k2; LCSC Part # (none) -> C2907117
- R106: renamed from R14; LCSC Part # (none) -> C26000; MPN (none) -> 0603WAJ0512T5E
- R108: renamed from R13; LCSC Part # (none) -> C103209; MPN (none) -> RTT03102JTP
- R109: renamed from R16; value 2k4 -> 2k2; LCSC Part # (none) -> C2907117
- R112: renamed from R3; LCSC Part # (none) -> C26000; MPN (none) -> 0603WAJ0512T5E
- R113: renamed from R4; value 2k4 -> 2k2; LCSC Part # (none) -> C2907117
- R114: renamed from R5; LCSC Part # (none) -> C26000; MPN (none) -> 0603WAJ0512T5E
- R115: renamed from R6; value 2k4 -> 2k2; LCSC Part # (none) -> C2907117
- R116: renamed from R7; LCSC Part # (none) -> C26000; MPN (none) -> 0603WAJ0512T5E
- R117: renamed from R8; LCSC Part # (none) -> C26000; MPN (none) -> 0603WAJ0512T5E
- R118: renamed from R9; LCSC Part # (none) -> C26000; MPN (none) -> 0603WAJ0512T5E
- R119: renamed from R10; LCSC Part # (none) -> C2907080; MPN (none) -> FRC0603P000 TS
- U101: renamed from U2; LCSC Part # (none) -> C5350818; MPN (none) -> IRF9358TRPBF
- U102: renamed from U1; LCSC Part # (none) -> C2959321
Connections:
- net +3V3: now also R107.1
- net GND: now also C101.2, Q102.3 (S), R111.2
- net PD_HPI: now also R107.2
- net VBUS: now also C102.1, C103.1, J101.A9 (VBUS), J101.B9 (VBUS), R106.1, U101.5 (D1), U101.6 (D1), U102.18 (VBUS_IN), C101.1; no longer C104.1, U101.1 (S2), U102.11 (VDC_OUT)
- net VBUS_MAX: now reaches R112.2, R113.1, U102.2 (VBUS_MAX)
- net ISNK_COARSE: now reaches R116.2, R117.1, U102.5 (ISNK_COARSE)
- net BUS_HEATSINK: now reaches U101.7 (D2), U101.8 (D2)
- net BUS_HEATSINK: now also C104.1, U102.11 (VDC_OUT), C109.1, C109.2, D102.1 (K), D102.2 (A), Q102.2 (D); no longer U101.3 (S1)
- net LED_FAULT: now reaches Q101.1 (G), R102.1, U102.9 (FAULT)
- net VBUS_EN: now reaches R108.2, U102.3
- net VBUS_MIN: now reaches R114.2, R115.1, U102.1 (VBUS_MIN)
- net CC2: now reaches J101.B5 (CC2), U102.14 (CC2)
- net CC1: now reaches J101.A5 (CC1), U102.15 (CC1)
- net SAFE: now reaches R109.2, U102.4
- net ISNK_FINE: now reaches R118.2, R119.1, U102.6 (ISNK_FINE)
- new net: U101.1 (S2), U101.3 (S1)
- new net: Q102.1 (G), R110.2, R111.1
- new net GATE_HEATER: R110.1
Other:
- added sheet Thermocouple (thermocouple.kicad_sch)
- sheet OLED Screen: file screen.kicad_sch -> OLEDScreen.kicad_sch
- note added: "HOT PLATE"
- note added: "SNUBBER"
- note removed: "DISEÑAR RED DE DESACOPLO!"
- note removed: "USAR PINES D+ y D- PARA MICRO¿?"
- moved on the sheet: C102, C103, C105, C106, C107, C108, D101, J101, Q101, R101, R102, R103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

Commit message: Pedido
Other:
- moved on the sheet: C105, C107, C108
