File: 01 - Board/KiCad/OLEDScreen.kicad_sch (KiCad schematic)
At the start: 21 parts, among them J4 OLED UG-9616TSWCG02, SW4 SW_Push, SW5 SW_Push, SW6 SW_Push

Commit message: Pedido
Other:
- title: (none) -> Hot Plate
Changed lines of the file:
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@@
 (kicad_sch (version 20230121) (generator eeschema)
   (paper "A4")
+  (title_block
+    (title "Hot Plate")
+    (date "2023-04-17")
+    (rev "AA")
+  )
   (junction (at 64.77 80.01) (diameter 0) (color 0 0 0 0)
   )
