File: 01 - Board/KiCad/thermocouple.kicad_sch (KiCad schematic)
At the start: 8 parts, among them U401 LM321LV

Commit message: Pedido
Other:
- title: (none) -> Hot Plate
Changed lines of the file:
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@@
 (kicad_sch (version 20230121) (generator eeschema)
   (paper "A4")
+  (title_block
+    (title "Hot Plate")
+    (date "2023-04-17")
+    (rev "AA")
+  )
   (junction (at 170.18 115.57) (diameter 0) (color 0 0 0 0)
   )
