File: 01 - KiCad/HotPlate.kicad_pcb (KiCad board)
At the start: 2 copper layers, 220 x 120 mm, 105 parts, among them J101 USB_C_Receptacle_PowerOnly_6P, J201 Conn_ARM_SWD_TagConnect_TC2030, J301 OLED UG-9616TSWCG02, Q101 2N7002, Q102 NMOS_ALT, SW301 SW_Push, SW302 SW_Push, SW303 SW_Push, U101 IRF9358TRPBF, U102 CYPD3177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

Commit message: SW 0.1 & updated Schematic
Connections:
- C305 pad 1: Net-(J301-VDDB) -> +3V3
- J301 pad 5: Net-(J301-VDDB) -> +3V3
Routing:
- net +3V3: track 295.8 -> 300.6 mm
- net Net-(J301-VDDB): track 3.06 -> 0.00 mm
