File: 01 - KiCad/MCU.kicad_sch (KiCad schematic)
At the start: 22 parts, among them J201 Conn_ARM_SWD_TagConnect_TC2030, U201 AP62300TWU, U202 STM32G030K8T6

Commit message: SW 0.1 & updated Schematic
Parts:
- C204, D102: now not fitted
Changed lines of the file:
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@@
   )
   (symbol (lib_id "Device:C") (at 90.17 82.55 0) (unit 1)
-    (in_bom yes) (on_board yes) (dnp no) (fields_autoplaced)
+    (in_bom yes) (on_board yes) (dnp yes) (fields_autoplaced)
     (property "Reference" "C204" (at 93.98 81.915 0)
       (effects (font (size 1.27 1.27)) (justify left))
@@
   )
   (symbol (lib_id "Device:D_Schottky") (at 217.17 120.65 270) (unit 1)
-    (in_bom yes) (on_board yes) (dnp no) (fields_autoplaced)
+    (in_bom yes) (on_board yes) (dnp yes) (fields_autoplaced)
     (property "Reference" "D102" (at 219.71 119.6975 90)
       (effects (font (size 1.27 1.27)) (justify left))
