File: 01 - KiCad/OLEDScreen.kicad_sch (KiCad schematic)
At the start: 21 parts, among them J4 OLED UG-9616TSWCG02, SW4 SW_Push, SW5 SW_Push, SW6 SW_Push

Commit message: SW 0.1 & updated Schematic
Connections:
- net +3V3: now also C2.1, J4.5 (VDDB)
Changed lines of the file:
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@@
   (junction (at 162.56 130.81) (diameter 0) (color 0 0 0 0)
+  )
+  (junction (at 189.23 102.87) (diameter 0) (color 0 0 0 0)
   )
   (junction (at 153.67 97.79) (diameter 0) (color 0 0 0 0)
@@
     (stroke (width 0) (type default))
   )
+  (wire (pts (xy 64.77 115.57) (xy 64.77 118.11))
+    (stroke (width 0) (type default))
+  )
+  (wire (pts (xy 64.77 161.29) (xy 64.77 162.56))
+    (stroke (width 0) (type default))
+  )
+  (wire (pts (xy 64.77 80.01) (xy 72.39 80.01))
+    (stroke (width 0) (type default))
+  )
+  (wire (pts (xy 162.56 97.79) (xy 162.56 107.95))
+    (stroke (width 0) (type default))
+  )
+  (wire (pts (xy 64.77 140.97) (xy 64.77 142.24))
+    (stroke (width 0) (type default))
+  )
+  (wire (pts (xy 217.17 82.55) (xy 217.17 83.82))
+    (stroke (width 0) (type default))
+  )
+  (wire (pts (xy 153.67 115.57) (xy 153.67 135.89))
+    (stroke (width 0) (type default))
+  )
+  (wire (pts (xy 229.87 82.55) (xy 217.17 82.55))
+    (stroke (width 0) (type default))
+  )
+  (wire (pts (xy 200.66 116.84) (xy 200.66 118.11))
+    (stroke (width 0) (type default))
+  )
+  (wire (pts (xy 64.77 114.3) (xy 64.77 115.57))
+    (stroke (width 0) (type default))
+  )
+  (wire (pts (xy 50.8 115.57) (xy 50.8 116.84))
+    (stroke (width 0) (type default))
+  )
+  (wire (pts (xy 217.17 78.74) (xy 217.17 80.01))
+    (stroke (width 0) (type default))
+  )
+  (wire (pts (xy 171.45 97.79) (xy 179.07 97.79))
+    (stroke (width 0) (type default))
+  )
+  (wire (pts (xy 153.67 97.79) (xy 153.67 107.95))
+    (stroke (width 0) (type default))
+  )
+  (wire (pts (xy 148.59 130.81) (xy 162.56 130.81))
+    (stroke (width 0) (type default))
+  )
+  (wire (pts (xy 189.23 102.87) (xy 229.87 102.87))
+    (stroke (width 0) (type default))
+  )
+  (wire (pts (xy 50.8 80.01) (xy 50.8 81.28))
+    (stroke (width 0) (type default))
+  )
+  (wire (pts (xy 64.77 151.13) (xy 64.77 153.67))
+    (stroke (width 0) (type default))
+  )
+  (wire (pts (xy 64.77 78.74) (xy 64.77 80.01))
+    (stroke (width 0) (type default))
+  )
+  (wire (pts (xy 64.77 69.85) (xy 64.77 71.12))
+    (stroke (width 0) (type default))
+  )
+  (wire (pts (xy 64.77 115.57) (xy 72.39 115.57))
+    (stroke (width 0) (type default))
+  )
+  (wire (pts (xy 64.77 151.13) (xy 50.8 151.13))
+    (stroke (width 0) (type default))
+  )
+  (wire (pts (xy 162.56 115.57) (xy 162.56 130.81))
+    (stroke (width 0) (type default))
+  )
+  (wire (pts (xy 220.98 113.03) (xy 229.87 113.03))
+    (stroke (width 0) (type default))
+  )
+  (wire (pts (xy 212.09 118.11) (xy 212.09 116.84))
+    (stroke (width 0) (type default))
+  )
+  (wire (pts (xy 189.23 101.6) (xy 189.23 102.87))
+    (stroke (width 0) (type default))
+  )
+  (wire (pts (xy 217.17 91.44) (xy 217.17 92.71))
+    (stroke (width 0) (type default))
+  )
+  (wire (pts (xy 64.77 115.57) (xy 50.8 115.57))
+    (stroke (width 0) (type default))
+  )
   (wire (pts (xy 179.07 97.79) (xy 229.87 97.79))
-    (stroke (width 0) (type default))
-  )
-  (wire (pts (xy 64.77 115.57) (xy 64.77 118.11))
-    (stroke (width 0) (type default))
-  )
-  (wire (pts (xy 64.77 161.29) (xy 64.77 162.56))
-    (stroke (width 0) (type default))
-  )
-  (wire (pts (xy 64.77 80.01) (xy 72.39 80.01))
-    (stroke (width 0) (type default))
-  )
-  (wire (pts (xy 162.56 97.79) (xy 162.56 107.95))
-    (stroke (width 0) (type default))
-  )
-  (wire (pts (xy 64.77 140.97) (xy 64.77 142.24))
-    (stroke (width 0) (type default))
-  )
-  (wire (pts (xy 217.17 82.55) (xy 217.17 83.82))
-    (stroke (width 0) (type default))
-  )
-  (wire (pts (xy 153.67 115.57) (xy 153.67 135.89))
-    (stroke (width 0) (type default))
-  )
-  (wire (pts (xy 229.87 82.55) (xy 217.17 82.55))
-    (stroke (width 0) (type default))
-  )
-  (wire (pts (xy 200.66 116.84) (xy 200.66 118.11))
-    (stroke (width 0) (type default))
-  )
-  (wire (pts (xy 64.77 114.3) (xy 64.77 115.57))
-    (stroke (width 0) (type default))
-  )
-  (wire (pts (xy 50.8 115.57) (xy 50.8 116.84))
-    (stroke (width 0) (type default))
-  )
-  (wire (pts (xy 217.17 78.74) (xy 217.17 80.01))
-    (stroke (width 0) (type default))
-  )
-  (wire (pts (xy 171.45 97.79) (xy 179.07 97.79))
-    (stroke (width 0) (type default))
-  )
-  (wire (pts (xy 153.67 97.79) (xy 153.67 107.95))
-    (stroke (width 0) (type default))
-  )
-  (wire (pts (xy 148.59 130.81) (xy 162.56 130.81))
-    (stroke (width 0) (type default))
-  )
-  (wire (pts (xy 189.23 102.87) (xy 229.87 102.87))
-    (stroke (width 0) (type default))
-  )
-  (wire (pts (xy 50.8 80.01) (xy 50.8 81.28))
-    (stroke (width 0) (type default))
-  )
-  (wire (pts (xy 64.77 151.13) (xy 64.77 153.67))
-    (stroke (width 0) (type default))
-  )
-  (wire (pts (xy 64.77 78.74) (xy 64.77 80.01))
-    (stroke (width 0) (type default))
-  )
-  (wire (pts (xy 64.77 69.85) (xy 64.77 71.12))
-    (stroke (width 0) (type default))
-  )
-  (wire (pts (xy 64.77 115.57) (xy 72.39 115.57))
-    (stroke (width 0) (type default))
-  )
-  (wire (pts (xy 64.77 151.13) (xy 50.8 151.13))
-    (stroke (width 0) (type default))
-  )
-  (wire (pts (xy 162.56 115.57) (xy 162.56 130.81))
-    (stroke (width 0) (type default))
-  )
-  (wire (pts (xy 220.98 113.03) (xy 229.87 113.03))
-    (stroke (width 0) (type default))
-  )
-  (wire (pts (xy 212.09 118.11) (xy 212.09 116.84))
-    (stroke (width 0) (type default))
-  )
-  (wire (pts (xy 217.17 91.44) (xy 217.17 92.71))
-    (stroke (width 0) (type default))
-  )
-  (wire (pts (xy 64.77 115.57) (xy 50.8 115.57))
     (stroke (width 0) (type default))
   )
@@
         )
       )
+    )
+  )
+  (symbol (lib_id "power:+3V3") (at 189.23 101.6 0) (unit 1)
+    (in_bom yes) (on_board yes) (dnp no)
+    (property "Reference" "#PWR015" (at 189.23 105.41 0)
+      (effects (font (size 1.27 1.27)) hide)
+    )
+    (property "Value" "+3V3" (at 193.04 100.33 0)
+      (effects (font (size 1.27 1.27)))
+    )
+    (property "Footprint" "" (at 189.23 101.6 0)
+      (effects (font (size 1.27 1.27)) hide)
+    )
+    (property "Datasheet" "" (at 189.23 101.6 0)
+      (effects (font (size 1.27 1.27)) hide)
+    )
+    (pin "1")
+    (instances
+      (project "HotPlate"
+        (path "/863ba709-7012-483f-92c6-07dcdce37e73"
+          (reference "#PWR015") (unit 1)
+        )
+        (path "/863ba709-7012-483f-92c6-07dcdce37e73/caded603-aabf-47a4-bf08-952390336771"
+          (reference "#PWR046") (unit 1)
+        )
+        (path "/863ba709-7012-483f-92c6-07dcdce37e73/ee61bde0-93c6-4775-b300-f7f2d61c8fcd"
+          (reference "#PWR0316") (unit 1)
+        )
+      )
